File: WLED_Controller_Board.kicad_sch (KiCad schematic)
At the start: 20 parts, among them IC1 SN74HCT125D, J1 Barrel_Jack, J2 FTDI Programmer, J3 WLED (VCC, DI, DI2, GND), J4 DHT11 / DHT22, SW1 Reset, SW2 Prog, U1 ESP-12E, U2 AMS1117-3.3

Commit message: Add files via upload
Change DHT VCC to 3.3V
Connections:
- net +3V3: now also J4.3 (Pin_3)
- net +5V: no longer J4.3 (Pin_3)
Changed lines of the file:
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@@
   (junction (at 147.32 87.63) (diameter 0) (color 0 0 0 0)
-  )
-  (junction (at 167.64 105.41) (diameter 0) (color 0 0 0 0)
   )
   (junction (at 101.6 33.02) (diameter 0) (color 0 0 0 0)
@@
   (no_connect (at 161.29 121.92))
   (no_connect (at 161.29 116.84))
-  (no_connect (at 161.29 114.3))
   (no_connect (at 133.35 119.38))
   (no_connect (at 133.35 121.92))
+  (no_connect (at 161.29 114.3))
   (wire (pts (xy 54.61 78.74) (xy 44.45 78.74))
     (stroke (width 0) (type default) (color 0 0 0 0))
@@
     (stroke (width 0) (type default) (color 0 0 0 0))
   )
-  (wire (pts (xy 229.87 127) (xy 229.87 105.41))
-    (stroke (width 0) (type default) (color 0 0 0 0))
-  )
   (wire (pts (xy 167.64 53.34) (xy 162.56 53.34))
     (stroke (width 0) (type default) (color 0 0 0 0))
@@
     (stroke (width 0) (type default) (color 0 0 0 0))
   )
-  (wire (pts (xy 167.64 105.41) (xy 229.87 105.41))
-    (stroke (width 0) (type default) (color 0 0 0 0))
-  )
   (wire (pts (xy 245.11 114.3) (xy 245.11 118.11))
     (stroke (width 0) (type default) (color 0 0 0 0))
@@
     (stroke (width 0) (type default) (color 0 0 0 0))
   )
+  (wire (pts (xy 229.87 118.11) (xy 229.87 127))
+    (stroke (width 0) (type default) (color 0 0 0 0))
+  )
   (wire (pts (xy 161.29 111.76) (xy 184.15 111.76))
     (stroke (width 0) (type default) (color 0 0 0 0))
   )
-  (wire (pts (xy 167.64 105.41) (xy 167.64 101.6))
+  (wire (pts (xy 167.64 101.6) (xy 167.64 109.22))
     (stroke (width 0) (type default) (color 0 0 0 0))
   )
@@
     (stroke (width 0) (type default) (color 0 0 0 0))
   )
+  (wire (pts (xy 214.63 110.49) (xy 214.63 118.11))
+    (stroke (width 0) (type default) (color 0 0 0 0))
+  )
   (wire (pts (xy 31.75 33.02) (xy 38.1 33.02))
     (stroke (width 0) (type default) (color 0 0 0 0))
@@
     (stroke (width 0) (type default) (color 0 0 0 0))
   )
+  (wire (pts (xy 214.63 118.11) (xy 229.87 118.11))
+    (stroke (width 0) (type default) (color 0 0 0 0))
+  )
   (wire (pts (xy 217.17 66.04) (xy 224.79 66.04))
     (stroke (width 0) (type default) (color 0 0 0 0))
@@
   )
   (wire (pts (xy 167.64 57.15) (xy 167.64 53.34))
-    (stroke (width 0) (type default) (color 0 0 0 0))
-  )
-  (wire (pts (xy 167.64 109.22) (xy 167.64 105.41))
     (stroke (width 0) (type default) (color 0 0 0 0))
   )
@@
     (pin "1")
   )
+  (symbol (lib_id "power:+3.3V") (at 214.63 110.49 0) (unit 1)
+    (in_bom yes) (on_board yes) (fields_autoplaced)
+    (property "Reference" "#PWR?" (id 0) (at 214.63 114.3 0)
+      (effects (font (size 1.27 1.27)) hide)
+    )
+    (property "Value" "+3.3V" (id 1) (at 214.63 105.41 0))
+    (property "Footprint" "" (id 2) (at 214.63 110.49 0)
+      (effects (font (size 1.27 1.27)) hide)
+    )
+    (property "Datasheet" "" (id 3) (at 214.63 110.49 0)
+      (effects (font (size 1.27 1.27)) hide)
+    )
+    (pin "1")
+  )
   (symbol (lib_id "Connector:Screw_Terminal_01x04") (at 46.99 105.41 270) (unit 1)
     (in_bom yes) (on_board yes) (fields_autoplaced)
@@
       (reference "#PWR08") (unit 1) (value "GND") (footprint "")
     )
+    (path "/673fbeed-5c07-4a8a-bf85-62824b76f4c9"
+      (reference "#PWR?") (unit 1) (value "+3.3V") (footprint "")
+    )
     (path "/24b2d1aa-9fb6-40fb-8d13-c8684874cbed"

Commit message: Add files via upload
Parts:
- added R8: 330Ω, Resistor_SMD:R_0603_1608Metric_Pad0.98x0.95mm_HandSolder, symbol Device:R
- C1, C2: footprint (none) -> Capacitor_SMD:C_0603_1608Metric_Pad1.08x0.95mm_HandSolder
- C3: footprint (none) -> Capacitor_THT:C_Radial_D10.0mm_H20.0mm_P5.00mm
- F1: footprint (none) -> Fuse:Fuseholder_Littelfuse_100_series_5x20mm
- IC1: footprint SOIC127P600X175-14N -> OwnLibary:SOIC127P600X175-14N
- J1: footprint (none) -> Connector_BarrelJack:BarrelJack_Wuerth_6941xx301002
- J2: footprint (none) -> Connector_PinHeader_2.54mm:PinHeader_1x05_P2.54mm_Horizontal
- J3: value WLED (VCC, DI, DI2, GND) -> WLED (VCC, DI, CI, GND); footprint (none) -> TerminalBlock_Phoenix:TerminalBlock_Phoenix_PT-1,5-4-3.5-H_1x04_P3.50mm_Horizontal
- J4: footprint (none) -> TerminalBlock_Phoenix:TerminalBlock_Phoenix_PT-1,5-3-3.5-H_1x03_P3.50mm_Horizontal
- R1, R2, R3, R4, R5, R6, R7: footprint (none) -> Resistor_SMD:R_0603_1608Metric_Pad0.98x0.95mm_HandSolder
- SW1, SW2: footprint (none) -> Button_Switch_SMD:SW_SPST_CK_RS282G05A3
Connections:
- net GPIO14: now reaches U1.5 (GPIO14)
- net GPIO14: now also IC1.5 (2A)
- net CLK: now reaches IC1.6 (2Y)
- net CLK: now also R8.2
- net at J3.3 (Pin_3), R6.1: no longer J3.2 (Pin_2)
- new net: J3.2 (Pin_2), R8.1
- no-connect marks 17 -> 14
Other:
- moved on the sheet: R6
